Commit message: package built working

File: dvrk_model/model/wsn_both_psms_rotated.urdf.xacro (robot description, xacro)
@@ -42,6 +42,5 @@
       <parent link="camera"/>
       <child link="davinci_endo"/>
-      <!--origin rpy="3.141593 0 0" xyz="0.00290 0 0.5"/-->
-      <origin rpy="3.141593 0 0" xyz="0.0029 0 0.5"/>
+      <origin rpy="3.14 0 0" xyz="0.0029 0 0.5"/>
   </joint>
   <link name="davinci_endo">
